File: daughter_board.kicad_sch (KiCad schematic)
At the start: 9 parts, among them J2 Conn_02x25_Odd_Even, SW1 SW_Push

Commit message: drc: updated symbols
Changed lines of the file:
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@@
 		(dnp no)
 		(fields_autoplaced yes)
-		(property "Reference" "#PWR?"
+		(property "Reference" "#PWR0223"
 			(at 175.26 132.08 0)
 			(effects
@@
 			(project "ceda"
 				(path "/12a6dbe3-008d-4c5b-88f6-9f1c816060be/4f1cc97c-1ae7-488a-96b4-ad54fee0fde4"
-					(reference "#PWR?")
+					(reference "#PWR0223")
 					(unit 1)
 				)
@@
 		(dnp no)
 		(fields_autoplaced yes)
-		(property "Reference" "#PWR?"
+		(property "Reference" "#PWR0210"
 			(at 40.64 74.93 0)
 			(effects
@@
 			(project "ceda"
 				(path "/12a6dbe3-008d-4c5b-88f6-9f1c816060be/4f1cc97c-1ae7-488a-96b4-ad54fee0fde4"
-					(reference "#PWR?")
+					(reference "#PWR0210")
 					(unit 1)
 				)
@@
 		(on_board yes)
 		(dnp no)
-		(property "Reference" "#PWR?"
+		(property "Reference" "#PWR0214"
 			(at 229.87 130.81 0)
 			(effects
@@
 			(project "ceda"
 				(path "/12a6dbe3-008d-4c5b-88f6-9f1c816060be/4f1cc97c-1ae7-488a-96b4-ad54fee0fde4"
-					(reference "#PWR?")
+					(reference "#PWR0214")
 					(unit 1)
 				)
@@
 		(dnp no)
 		(fields_autoplaced yes)
-		(property "Reference" "#PWR?"
+		(property "Reference" "#PWR0208"
 			(at 160.02 26.67 0)
 			(effects
@@
 			(project "ceda"
 				(path "/12a6dbe3-008d-4c5b-88f6-9f1c816060be/4f1cc97c-1ae7-488a-96b4-ad54fee0fde4"
-					(reference "#PWR?")
+					(reference "#PWR0208")
 					(unit 1)
 				)
@@
 		(dnp no)
 		(fields_autoplaced yes)
-		(property "Reference" "#PWR?"
+		(property "Reference" "#PWR0212"
 			(at 60.96 74.93 0)
 			(effects
@@
 			(project "ceda"
 				(path "/12a6dbe3-008d-4c5b-88f6-9f1c816060be/4f1cc97c-1ae7-488a-96b4-ad54fee0fde4"
-					(reference "#PWR?")
-					(unit 1)
-				)
+					(reference "#PWR0212")
+					(unit 1)
+				)
