File: video_memory.kicad_sch (KiCad schematic)
At the start: 22 parts, among them J11 74LS245, J9 uPD446, K15 7417, U2 74LS10

Commit message: Edited some notes
Other:
- note added: "~{RD|WR}. Can't use ~{IOREQ} because WR is asserted one clock cycle later."
- note removed: "Active high Memory enable"
- note removed: "~{RD|WR}. Why not ~{IOREQ}? Nice question..."
Changed lines of the file:
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@@
   )
   (text "Character and attribute RAM can be concurrently\naddressed by Z80 and CRTC:\n- CRTC enables both RAMs during positive pulses\nof video main clock (1.875MHz).\n- Z80 selectively enables each RAM IC through a\nbank switch signal."
-    (at 229.87 275.59 0)
+    (at 308.61 175.26 0)
     (effects (font (size 1.27 1.27)) (justify left bottom))
   )
-  (text "Bank Switching for uPD446 RAM chips" (at 138.43 154.94 0)
-    (effects (font (size 2.54 2.54)) (justify left bottom))
+  (text "Bank Switching for uPD446 RAM chips" (at 308.61 160.02 0)
+    (effects (font (size 3 3) (thickness 0.6) bold) (justify left bottom))
   )
-  (text "~{RD|WR}. Why not ~{IOREQ}?\nNice question..." (at 120.65 215.9 0)
+  (text "~{RD|WR}. Can't use ~{IOREQ}\nbecause WR is asserted\none clock cycle later."
+    (at 120.65 215.9 0)
     (effects (font (size 1.27 1.27)) (justify left bottom))
   )
@@
   )
   (text "Z80 video memory access request is generated as follows:\n- is immediately asserted when /MREQ = 0 and address\nfalls in video memory address space (0xD000).\n- the deassertion is syncronized with video main clock.\n\nPlease note that code cannot be executed from video memory\nsince, if M1 is asserted, the access request is ignored.\nNo memory IC is selected if someone tries to fetch code from\nvideo memory address space!"
-    (at 331.47 250.19 0)
+    (at 308.61 196.85 0)
     (effects (font (size 1.27 1.27)) (justify left bottom))
   )
-  (text "Active high Memory enable" (at 190.5 194.31 0)
-    (effects (font (size 1.27 1.27)) (justify right bottom))
-  )
   (text "Video\n RAM" (at 166.37 43.18 0)

Commit message: Notes in kicad's sheet text blocks
Other:
- company: (none) -> Logic Systems Int'l Inc
- title: (none) -> CEDA - Sanco 8003 schematics
Changed lines of the file:
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@@
 (kicad_sch (version 20230121) (generator eeschema)
   (paper "A3")
+  (title_block
+    (title "CEDA - Sanco 8003 schematics")
+    (rev "05")
+    (company "Logic Systems Int'l Inc")
+    (comment 1 "reversed by RetrOfficina - retrofficina.glgprograms.it")
+    (comment 3 "Handle the concurrent access to video memory by the CPU and the CRTC")
+    (comment 4 "Video Memory Management")
+  )
   (junction (at 118.11 240.03) (diameter 0) (color 0 0 0 0)
   )

Commit message: Upgrade to KiCAD 9.0
Parts:
- renumbered K15 to UC2, E13 to UE13, E14 to UE14, E15 to UE15, E16 to UE16, F10 to UF10, F11 to UF11, F12 to UF12, F13 to UF13, F14 to UF14, F16 to UF16, F8 to UF8, F9 to UF9, H1 to UH1, H15 to UH15, H8H10 to UH8, J11 to UJ11, J9 to UJ9, U2 to UK14
Connections:
- net +5V: now also UH15.13 (~{R}); no longer UH15.1 (~{R})
- net half_pxclk: now also UH15.11 (C); no longer UH15.3 (C)
- net quart_pxclk: now also UH15.12 (D); no longer UH15.2 (D)
- net at UE14.12 (D): now also UH1.10; no longer UH1.2
- net at UE13.6, UF13.10, UF13.5: now also UH15.10 (~{S}); no longer UH15.4 (~{S})
- net at L3.8: now also UH1.11; no longer UH1.1
- net at UE16.10: now also UH15.9 (Q); no longer UH15.5 (Q)

Commit message: drc: corrections in net names
Changed lines of the file:
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@@
+		)
+	)
+	(label "vmem[10..0]"
+		(at 113.03 66.04 0)
+		(effects
+			(font
+				(size 1.27 1.27)
+			)
+			(justify left bottom)
 		)
 	)

Commit message: drc: fixed labels
Connections:
- net ~{RD|WR}: now reaches L3.8, UH1.11
- net MEM_WR renamed ~{MEM_WR}
- net MREQ renamed ~{MREQ}
Other:
- note added: "~{RD|WR}. Can't use ~{IORQ} because WR is asserted one clock cycle later."
- note removed: "~{RD|WR}. Can't use ~{IOREQ} because WR is asserted one clock cycle later."
Changed lines of the file:
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@@
 		)
 	)
-	(text "~{RD|WR}. Can't use ~{IOREQ}\nbecause WR is asserted\none clock cycle later."
+	(text "~{RD|WR}. Can't use ~{IORQ}\nbecause WR is asserted\none clock cycle later."
 		(exclude_from_sim no)
 		(at 120.65 215.9 0)
@@
 	)
 	(junction
+		(at 124.46 218.44)
+		(diameter 0)
+		(color 0 0 0 0)
+	)
+	(junction
 		(at 97.79 129.54)
 		(diameter 0)
@@
 	(wire
 		(pts
+			(xy 124.46 218.44) (xy 120.65 218.44)
+		)
+		(stroke
+			(width 0)
+			(type default)
+		)
+	)
+	(wire
+		(pts
 			(xy 74.93 237.49) (xy 88.9 237.49)
 		)
@@
 	(wire
 		(pts
+			(xy 124.46 220.98) (xy 125.73 220.98)
+		)
+		(stroke
+			(width 0)
+			(type default)
+		)
+	)
+	(wire
+		(pts
 			(xy 280.67 107.95) (xy 295.91 107.95)
 		)
@@
 	(wire
 		(pts
+			(xy 124.46 218.44) (xy 124.46 220.98)
+		)
+		(stroke
+			(width 0)
+			(type default)
+		)
+	)
+	(wire
+		(pts
 			(xy 335.28 40.64) (xy 321.31 40.64)
 		)
@@
 	(wire
 		(pts
-			(xy 142.24 218.44) (xy 120.65 218.44)
+			(xy 142.24 218.44) (xy 124.46 218.44)
 		)
 		(stroke
@@
 	(wire
 		(pts
-			(xy 157.48 220.98) (xy 166.37 220.98)
+			(xy 165.1 220.98) (xy 166.37 220.98)
 		)
 		(stroke
@@
 		)
 	)
-	(label "MUXSEL"
-		(at 157.48 220.98 0)
-		(effects
-			(font
-				(size 1.27 1.27)
-			)
-			(justify left bottom)
-		)
-	)
 	(label "vmem9"
 		(at 87.63 154.94 0)
@@
 		)
 	)
+	(global_label "~{RD|WR}"
+		(shape input)
+		(at 125.73 220.98 0)
+		(fields_autoplaced yes)
+		(effects
+			(font
+				(size 1.27 1.27)
+			)
+			(justify left)
+		)
+		(property "Intersheetrefs" "${INTERSHEET_REFS}"
+			(at 135.1861 220.98 0)
+			(effects
+				(font
+					(size 1.27 1.27)
+				)
+				(justify left)
+				(hide yes)
+			)
+		)
+	)
+	(global_label "~{CRTC_CLK}"
+		(shape input)
+		(at 165.1 220.98 180)
+		(fields_autoplaced yes)
+		(effects
+			(font
+				(size 1.27 1.27)
+			)
+			(justify right)
+		)
+		(property "Intersheetrefs" "${INTERSHEET_REFS}"
+			(at 152.8015 220.98 0)
+			(effects
+				(font
+					(size 1.27 1.27)
+				)
+				(justify right)
+				(hide yes)
+			)
+		)
+	)
 	(global_label "~{RESET}"
 		(shape input)
@@
 		)
 	)
-	(global_label "MREQ"
+	(global_label "~{MREQ}"
 		(shape input)
 		(at 54.61 240.03 180)
@@
 		)
 	)
-	(global_label "MEM_WR"
+	(global_label "~{MEM_WR}"
 		(shape input)
 		(at 270.51 227.33 180)
@@
 		)
 	)
-	(global_label "MEM_WR"
+	(global_label "~{MEM_WR}"
 		(shape input)
 		(at 323.85 60.96 0)

Commit message: Assigned default footprints to ICs
Parts:
- UC2, UE13, UE14, UE15, UE16, UF13, UF14, UF16, UH1, UH15, UK14: footprint (none) -> Package_DIP:DIP-14_W7.62mm
- UF10, UF8, UF9: footprint (none) -> Package_DIP:DIP-16_W7.62mm
- UF11, UF12, UJ11: footprint (none) -> Package_DIP:DIP-20_W7.62mm
- UH8, UJ9: footprint (none) -> Package_DIP:DIP-24_W7.62mm
Changed lines of the file:
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@@
 			)
 		)
-		(property "Footprint" ""
+		(property "Footprint" "Package_DIP:DIP-14_W7.62mm"
 			(at 203.2 167.64 0)
 			(effects
@@
 			)
 		)
-		(property "Footprint" ""
+		(property "Footprint" "Package_DIP:DIP-20_W7.62mm"
 			(at 220.98 114.3 0)
 			(effects
@@
 			)
 		)
-		(property "Footprint" ""
+		(property "Footprint" "Package_DIP:DIP-14_W7.62mm"
 			(at 182.88 165.1 0)
 			(effects
@@
 			)
 		)
-		(property "Footprint" ""
+		(property "Footprint" "Package_DIP:DIP-14_W7.62mm"
 			(at 173.99 220.98 0)
 			(effects
@@
 			)
 		)
-		(property "Footprint" ""
+		(property "Footprint" "Package_DIP:DIP-14_W7.62mm"
 			(at 260.35 165.1 0)
 			(effects
@@
 			)
 		)
-		(property "Footprint" ""
+		(property "Footprint" "Package_DIP:DIP-14_W7.62mm"
 			(at 283.21 134.62 0)
 			(effects
@@
 			)
 		)
-		(property "Footprint" ""
+		(property "Footprint" "Package_DIP:DIP-14_W7.62mm"
 			(at 161.29 260.35 0)
 			(effects
@@
 			)
 		)
-		(property "Footprint" ""
+		(property "Footprint" "Package_DIP:DIP-14_W7.62mm"
 			(at 67.31 237.49 0)
 			(effects
@@
 			)
 		)
-		(property "Footprint" ""
+		(property "Footprint" "Package_DIP:DIP-24_W7.62mm"
 			(at 168.91 24.13 0)
 			(effects
@@
 			)
 		)
-		(property "Footprint" ""
+		(property "Footprint" "Package_DIP:DIP-14_W7.62mm"
 			(at 281.94 224.79 0)
 			(effects
@@
 			)
 		)
-		(property "Footprint" ""
+		(property "Footprint" "Package_DIP:DIP-16_W7.62mm"
 			(at 74.93 102.87 0)
 			(effects
@@
 			)
 		)
-		(property "Footprint" ""
+		(property "Footprint" "Package_DIP:DIP-20_W7.62mm"
 			(at 308.61 50.8 0)
 			(effects
@@
 			)
 		)
-		(property "Footprint" ""
+		(property "Footprint" "Package_DIP:DIP-24_W7.62mm"
 			(at 168.91 88.9 0)
 			(effects
@@
 			)
 		)
-		(property "Footprint" ""
+		(property "Footprint" "Package_DIP:DIP-20_W7.62mm"
 			(at 308.61 105.41 0)
 			(effects
@@
 			)
 		)
-		(property "Footprint" ""
+		(property "Footprint" "Package_DIP:DIP-14_W7.62mm"
 			(at 133.35 237.49 0)
 			(effects
@@
 			)
 		)
-		(property "Footprint" ""
+		(property "Footprint" "Package_DIP:DIP-14_W7.62mm"
 			(at 260.35 187.96 0)
 			(effects
@@
 			)
 		)
-		(property "Footprint" ""
+		(property "Footprint" "Package_DIP:DIP-14_W7.62mm"
 			(at 203.2 185.42 0)
 			(effects
@@
 			)
 		)
-		(property "Footprint" ""
+		(property "Footprint" "Package_DIP:DIP-16_W7.62mm"
 			(at 74.93 162.56 0)
 			(effects
@@
 			)
 		)
-		(property "Footprint" ""
+		(property "Footprint" "Package_DIP:DIP-14_W7.62mm"
 			(at 36.83 196.85 0)
 			(effects
@@
 			)
 		)
-		(property "Footprint" ""
+		(property "Footprint" "Package_DIP:DIP-16_W7.62mm"
 			(at 74.93 43.18 0)
 			(effects
@@
 			)
 		)
-		(property "Footprint" ""
+		(property "Footprint" "Package_DIP:DIP-14_W7.62mm"
 			(at 97.79 240.03 0)
 			(effects
@@
 			)
 		)
-		(property "Footprint" ""
+		(property "Footprint" "Package_DIP:DIP-14_W7.62mm"
 			(at 149.86 218.44 0)
 			(effects
@@
 			)
 		)
-		(property "Footprint" ""
+		(property "Footprint" "Package_DIP:DIP-14_W7.62mm"
 			(at 302.26 212.09 0)
 			(effects
@@
 			)
 		)
-		(property "Footprint" ""
+		(property "Footprint" "Package_DIP:DIP-14_W7.62mm"
 			(at 250.19 212.09 0)
 			(effects
@@
 			)
 		)
-		(property "Footprint" ""
+		(property "Footprint" "Package_DIP:DIP-14_W7.62mm"
 			(at 142.24 257.81 0)
 			(effects
@@
 			)
 		)
-		(property "Footprint" ""
+		(property "Footprint" "Package_DIP:DIP-14_W7.62mm"
 			(at 93.98 257.81 0)
 			(effects
@@
 			)
 		)
-		(property "Footprint" ""
+		(property "Footprint" "Package_DIP:DIP-14_W7.62mm"
 			(at 236.22 196.85 0)
 			(effects

Commit message: Fixed packages
Parts:
- UH8, UJ9: footprint Package_DIP:DIP-24_W7.62mm -> Package_DIP:DIP-24_W15.24mm
Changed lines of the file:
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@@
 			)
 		)
-		(property "Footprint" "Package_DIP:DIP-24_W7.62mm"
+		(property "Footprint" "Package_DIP:DIP-24_W15.24mm"
 			(at 168.91 24.13 0)
 			(effects
@@
 			)
 		)
-		(property "Footprint" "Package_DIP:DIP-24_W7.62mm"
+		(property "Footprint" "Package_DIP:DIP-24_W15.24mm"
 			(at 168.91 88.9 0)
 			(effects
