File: ceda.kicad_pcb (KiCad board)
At the start: 4 copper layers, 302.3 x 218.4 mm, 112 parts, among them K9 4164, SW1 SW_DIP_x08, U15 L78L05_TO92

Commit message: pcb: added more traces
Connections:
- UE15 pad 2: MEM_OE -> ~{MEM_OE}
- UE15 pad 4: MEM_OE -> ~{MEM_OE}
- UH1 pad 6: /MainMemoryManagement/MREQ -> MREQ
- UJ11 pad 1: MEM_OE -> ~{MEM_OE}
- UK14 pad 13: ~{MREQ} -> MREQ
- UL4 pad 9: /MainMemoryManagement/MREQ -> MREQ
Routing:
- net ~{D000_CS}: track 54.6 -> 337.9 mm, vias 1 -> 3
- net MREQ: track 0.00 -> 282.6 mm, vias 0 -> 4
- net (no net): track 0.00 -> 268.6 mm, vias 0 -> 3
- net disptmg_reg: track 55.7 -> 288.0 mm, vias 2 -> 4
- net Net-(UB5B-Q): track 0.00 -> 223.1 mm, vias 0 -> 1
- net Net-(UB6A-~{R}): track 0.00 -> 221.0 mm, vias 0 -> 2
- net Net-(UB5A-Q): track 0.00 -> 220.9 mm, vias 0 -> 1
- net ~{PerrorReset_CS}: track 0.00 -> 212.9 mm, vias 0 -> 3
- net /VideoGeneration/~{cudisp_reg}: track 15.1 -> 221.5 mm, vias 0 -> 2
- net D2: track 314.3 -> 513.8 mm, vias 9 -> 13
- net D0: track 324.2 -> 523.4 mm, vias 11 -> 14
- net Net-(UL9A-~{R}): track 0.00 -> 196.0 mm, vias 0 -> 2
- net ~{MEM_OE}: track 92.3 -> 284.0 mm, vias 2 -> 3
- net ~{RD}: track 244.9 -> 410.2 mm, vias 4 -> 6
- net Net-(UB8B-~{R}): track 22.8 -> 180.3 mm, vias 0 -> 2
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