File: ceda.kicad_pcb (KiCad board)
At the start: 4 copper layers, 302.3 x 218.4 mm, 253 parts, among them J1 Conn_02x18_Odd_Even, J2 Conn_02x25_Odd_Even, J3 Conn_02x06_Odd_Even, J4 MAINCLK, J5 SIOCLK, J6 EXBUS, J7 POWER, SW1 SW_DIP_x08, U15 L78L05_TO92

Commit message: pcb: fixed traces
Parts:
- added C28: 330p, Capacitor_THT:C_Disc_D4.3mm_W1.9mm_P5.00mm, F.Cu at (48.3, 190.4)
- moved C105 2.54 mm to (287.0, 66.0)
- moved C7778 2.54 mm to (27.9, 25.4)
- moved C104 2.54 mm to (12.7, 12.7)
- moved C6 0.06 mm to (22.9, 17.8)
Connections:
- J2 pad 50: SER_10 -> -12V
- UB4 pad 7: (no net) -> GND
- UB4 pad 9: (no net) -> +5VL
- UC15 pad 12: unconnected-(UC15-Pad12) -> Net-(C28-Pad2)
- UD15 pad 1: (no net) -> -12V
- UD15 pad 14: (no net) -> +12V
- UD15 pad 7: (no net) -> GND
- UD16 pad 1: (no net) -> -12V
- UD16 pad 14: (no net) -> +12V
- UD16 pad 7: (no net) -> GND
Routing:
- net -12V: track 0.00 -> 299.7 mm
- net +12V: track 468.3 -> 531.5 mm, vias 0 -> 2
- net Net-(C28-Pad2): track 0.00 -> 26.4 mm
- net (no net): track 17.8 -> 0.00 mm
- net Net-(U15-VI): track 183.9 -> 188.9 mm
- net Net-(C105-Pad1): track 47.9 -> 45.4 mm
- net ~{RD}: track 487.0 -> 484.9 mm
- net +5VL: track 146.6 -> 148.6 mm
- net unconnected-(UA6-TC-Pad15): track 1.78 -> 0.00 mm
- net PRINTER_22: track 128.4 -> 130.2 mm
- net D7: track 567.0 -> 565.5 mm
- net A13: track 165.6 -> 164.4 mm
- net A12: track 217.5 -> 216.5 mm
- net /FloppyDiskController/~{DIRECTION}: track 28.8 -> 29.6 mm
- net PRINTER_24: track 121.1 -> 121.9 mm
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