File: ceda.kicad_pcb (KiCad board)
At the start: 4 copper layers, 302.3 x 218.4 mm, 262 parts, among them J1 Conn_02x18_Odd_Even, J2 Conn_02x25_Odd_Even, J3 Conn_02x06_Odd_Even, J4 MAINCLK, J5 SIOCLK, J6 EXBUS, J7 POWER, SW1 SW_DIP_x08, U15 L78L05_TO92

Commit message: pcb: proper symbols for MAP and MAINCLK
Parts:
- removed MAP1: SolderJumper_2_Open, Connector_PinHeader_2.54mm:PinHeader_2x01_P2.54mm_Vertical
- removed MAP2, MAP3: SolderJumper_2_Bridged, Connector_PinHeader_2.54mm:PinHeader_2x01_P2.54mm_Vertical
- added JP4: MAP, Ceda:MAP, F.Cu at (274.3, 8.89)
- J4: footprint Connector_PinHeader_2.54mm:PinHeader_2x02_P2.54mm_Vertical -> Ceda:MAINCLK
- moved J4 1.80 mm to (6.35, 85.1)
